File: Board master-slave/master/master.kicad_sch (KiCad schematic)
At the start: 131 parts, among them J1 USB_C_16P, J11 PZEM, J12 FS300A, J15 MAX31865, J16 PH_SENSOR, J2 JackDC - 12V, J3 Conn_01x04, J4 Y26, J5 Conn_01x03, J6 TDS, J7 SHT30, J8 Conn_01x06, J9 JackDC - 12V, Q1 AOD407, Q10 S8050, Q11 S8050, Q4 S8050, Q5 SS8050, Q6 S8050, Q7 S8050, Q8 SS8050, Q9 S8050, SW1 SW_Push, SW2 SW_Push, U1 ESP32-WROOM-32UE, U2 TPS5430DDA 12V->5V, U3 TPS5430DDA 12V->3.3V, U4 CH340C, U5 STM32F103C8T6, Y1 8MHz, Y2 Crystal_GND23

Commit message: Di day mach nguon
Parts:
- removed J9: JackDC - 12V, Connector_BarrelJack:BarrelJack_Horizontal, symbol Connector:Barrel_Jack_Switch
Changed lines of the file:
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@@
-	)
-	(symbol
-		(lib_id "Connector:Barrel_Jack_Switch")
-		(at -25.4 -135.89 0)
-		(unit 1)
-		(body_style 1)
-		(exclude_from_sim no)
-		(in_bom yes)
-		(on_board yes)
-		(in_pos_files yes)
-		(dnp no)
-		(fields_autoplaced yes)
-		(property "Reference" "J9"
-			(at -25.4 -144.78 0)
-			(hide yes)
-			(show_name no)
-			(do_not_autoplace no)
-			(effects
-				(font
-					(size 1.27 1.27)
-				)
-			)
-		)
-		(property "Value" "JackDC - 12V"
-			(at -25.4 -142.24 0)
-			(show_name no)
-			(do_not_autoplace no)
-			(effects
-				(font
-					(size 1.27 1.27)
-				)
-			)
-		)
-		(property "Footprint" "Connector_BarrelJack:BarrelJack_Horizontal"
-			(at -24.13 -134.874 0)
-			(hide yes)
-			(show_name no)
-			(do_not_autoplace no)
-			(effects
-				(font
-					(size 1.27 1.27)
-				)
-			)
-		)
-		(property "Datasheet" ""
-			(at -24.13 -134.874 0)
-			(hide yes)
-			(show_name no)
-			(do_not_autoplace no)
-			(effects
-				(font
-					(size 1.27 1.27)
-				)
-			)
-		)
-		(property "Description" "DC Barrel Jack with an internal switch"
-			(at -25.4 -135.89 0)
-			(hide yes)
-			(show_name no)
-			(do_not_autoplace no)
-			(effects
-				(font
-					(size 1.27 1.27)
-				)
-			)
-		)
-		(pin "3"
-		)
-		(pin "1"
-		)
-		(pin "2"
-		)
-		(instances
-			(project "master"
-				(path "/d2cec5e8-356f-4709-9dd3-ca1a140b7306"
-					(reference "J9")
-					(unit 1)
-				)
-			)
-		)
 	)
 	(symbol
