File: Board master-slave/master/master.kicad_pcb (KiCad board)
At the start: 2 copper layers, 135 parts, among them J1 USB_C_16P, J11 PZEM, J12 FS300A, J15 MAX31865, J16 PH_SENSOR, J2 JackDC - 12V, J3 Conn_01x04, J4 Y26, J5 Conn_01x03, J6 TDS, J7 SHT30, J8 Conn_01x06, Q1 AOD407, Q10 S8050, Q11 S8050, Q4 S8050, Q5 SS8050, Q6 S8050, Q7 S8050, Q8 SS8050, Q9 S8050, SW1 SW_Push, SW2 SW_Push, U1 ESP32-WROOM-32UE, U2 TPS5430DDA 12V->5V, U3 TPS5430DDA 12V->3.3V, U4 CH340C, U5 STM32F103C8T6, Y1 8MHz, Y2 Crystal_GND23

Commit message: Update di day
Parts:
- moved C27 1.81 mm to (218.8, 85.7)
- moved R19 1.81 mm to (227.3, 85.6)
- moved Y2 1.81 mm to (220.8, 91.5)
- moved C26 1.81 mm to (222.7, 85.7)
- moved Y1 1.81 mm to (226.9, 89.7)
- moved C25 1.59 mm to (229.9, 91.2), turned to -90 degrees
- moved C24 1.28 mm to (229.8, 86.9)
- turned D8 to 180 degrees
Routing:
- net /3.3V: track 84.6 -> 205.4 mm, vias 0 -> 1
- net /3.3V_STM: track 0.00 -> 73.2 mm, vias 0 -> 4
- net /PB13/RELAY2_CTRL: track 0.00 -> 55.0 mm, vias 0 -> 1
- net /PB12/RELAY1_CTRL: track 0.00 -> 54.4 mm, vias 0 -> 1
- net /PA5/PH_ADC: track 0.00 -> 53.2 mm
- net /PB14/RELAY3_CTRL: track 0.00 -> 52.0 mm, vias 0 -> 1
- net /PB1/TDS_ADC: track 0.00 -> 49.7 mm, vias 0 -> 2
- net /PB15/RELAY4_CTRL: track 0.00 -> 49.2 mm, vias 0 -> 1
- net /PA12/MAX31865_CS: track 0.00 -> 48.3 mm, vias 0 -> 1
- net /PA11/MAX31865_MOSI: track 0.00 -> 48.2 mm, vias 0 -> 3
- net /TX2: track 0.00 -> 47.1 mm, vias 0 -> 2
- net /PA7/MAX31865_MISO: track 0.00 -> 46.9 mm, vias 0 -> 3
- net /RX2: track 0.00 -> 46.8 mm, vias 0 -> 2
- net /PA6/MAX31865_SCK: track 0.00 -> 44.7 mm, vias 0 -> 1
- net /RESET: track 0.00 -> 42.4 mm, vias 0 -> 1
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