File: Board master-slave/master/master.kicad_pcb (KiCad board)
At the start: 4 copper layers, 135 parts, among them J1 USB_C_16P, J11 PZEM, J12 FS300A, J15 MAX31865, J16 PH_SENSOR, J3 Conn_01x04, J4 Y26, J5 SRC-RELAY, J6 TDS, J7 SHT30, J8 RELAY-CONTROL, J9 JackDC - 12V, Q1 AOD407, Q10 S8050, Q11 S8050, Q4 S8050, Q5 SS8050, Q6 S8050, Q7 S8050, Q8 SS8050, Q9 S8050, SW1 SW_Push, SW2 SW_Push, U1 ESP32-WROOM-32UE, U2 TPS5430DDA 12V->5V, U3 TPS5430DDA 12V->3.3V, U4 CH340C, U5 STM32F103C8T6, Y1 8MHz, Y2 Crystal_GND23

Commit message: Di day mach nguon
Parts:
- removed J9: JackDC - 12V, Connector_BarrelJack:BarrelJack_Horizontal
- added J2: JackDC - 12V, Connector_BarrelJack:BarrelJack_Horizontal, F.Cu at (270.5, 24.0)
- J5: value SRC-RELAY -> Conn_01x03
- J8: value RELAY-CONTROL -> Conn_01x06
- SWD1: value JLINK -> Conn_01x04
- moved REF** 20.2 mm to (239.5, 79.5)
- moved D2 15.6 mm to (266.6, 45.4), turned to 0 degrees
- moved D5 15.5 mm to (266.8, 32.8), turned to 0 degrees
- moved R20 8.49 mm to (229.4, 58.5)
- moved JP2x32.1 8.49 mm to (226.5, 60.0)
- moved R22 8.49 mm to (221.0, 58.7)
- moved D18 1.47 mm to (234.3, 27.1)
- moved D19 1.47 mm to (229.1, 27.1)
- moved D20 1.47 mm to (224.1, 27.1)
- moved J3 1.47 mm to (234.1, 18.1)
- moved Q1 1.21 mm to (261.0, 21.0), turned to 180 degrees
- moved L1 0.81 mm to (257.2, 48.5)
- moved F2 0.67 mm to (272.0, 14.9)
- moved C2 0.57 mm to (265.8, 51.0), turned to 90 degrees
- moved J1 0.51 mm to (204.7, 16.5)
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Routing:
- net /5V: track 0.00 -> 136.8 mm, vias 0 -> 14
- net /Vin: track 0.00 -> 115.4 mm, vias 0 -> 4
- net /3.3V: track 0.00 -> 40.3 mm
- net Net-(U2-VSENSE): track 0.00 -> 25.6 mm
- net Net-(U3-VSENSE): track 0.00 -> 24.6 mm
- net Net-(D2-K): track 0.00 -> 20.9 mm
- net Net-(D5-K): track 0.00 -> 20.0 mm
- net Net-(F2-Pad1): track 0.00 -> 14.7 mm, vias 0 -> 1
- net Net-(D21-K): track 0.00 -> 13.3 mm
- net Net-(D22-K): track 0.00 -> 13.0 mm
- net Net-(D3-K): track 0.00 -> 10.6 mm
- net Net-(D3-A): track 0.00 -> 9.11 mm
- net Net-(D18-K): track 0.00 -> 7.06 mm
- net Net-(D19-K): track 0.00 -> 6.99 mm
- net Net-(D20-K): track 0.00 -> 6.95 mm
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Other:
- copper layers 4 -> 2

Commit message: pcb layout 1
Parts:
- moved J7 71.3 mm to (188.8, 79.0), turned to 180 degrees
- moved J12 43.3 mm to (213.5, 108.1), turned to 90 degrees
- moved R23 35.6 mm to (219.2, 103.7), turned to 180 degrees
- moved J6 34.9 mm to (249.8, 108.2), turned to 90 degrees
- moved J16 7.53 mm to (260.4, 108.2)
- moved D17 5.33 mm to (200.0, 58.6), turned to 180 degrees
- moved R38 4.39 mm to (224.3, 104.3)
- moved R39 4.39 mm to (231.9, 100.7)
- moved J4 3.40 mm to (223.6, 108.2)
- moved R28 2.80 mm to (204.2, 56.1), turned to 180 degrees
- moved R12 2.22 mm to (211.2, 16.7)
- moved C4 1.84 mm to (195.0, 56.1), turned to 180 degrees
- moved C9 1.79 mm to (194.9, 58.3), turned to 180 degrees
- moved R24 1.71 mm to (244.9, 100.3)
- moved R25 1.71 mm to (237.3, 104.2)
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Routing:
- net /5V: track 136.8 -> 199.3 mm
- net /3.3V: track 40.3 -> 84.6 mm
- net /IO0: track 0.00 -> 35.4 mm, vias 0 -> 2
- net /EN: track 0.00 -> 27.6 mm
- net Net-(Q5-E): track 0.00 -> 17.1 mm
- net Net-(Q8-E): track 0.00 -> 13.8 mm
- net /3V3_ESP: track 0.00 -> 11.7 mm
- net Net-(U4-UD-): track 0.00 -> 9.36 mm, vias 0 -> 2
- net Net-(Q5-B): track 0.00 -> 9.00 mm, vias 0 -> 2
- net /CC1: track 0.00 -> 6.72 mm
- net /CC2: track 0.00 -> 6.36 mm
- net Net-(U4-UD+): track 0.00 -> 5.87 mm
- net Net-(J11-Pin_3): track 0.00 -> 5.30 mm
- net Net-(Q8-B): track 0.00 -> 4.82 mm, vias 0 -> 2
- net /PA1/FLOW_SIG: track 0.00 -> 4.72 mm
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
Commit message: pcb update
Parts:
- moved C21 1.34 mm to (231.5, 81.2), turned to 90 degrees
- turned D8 to 180 degrees
Routing:
- net /3.3V: track 84.6 -> 241.1 mm, vias 0 -> 1
- net /TX2: track 0.00 -> 47.0 mm, vias 0 -> 2
- net /RX2: track 0.00 -> 46.8 mm, vias 0 -> 2
- net /3.3V_STM: track 0.00 -> 46.4 mm
- net /3V3_ESP: track 11.7 -> 57.0 mm, vias 0 -> 1
- net /RESET: track 0.00 -> 42.0 mm, vias 0 -> 1
- net Net-(U4-RXD): track 0.00 -> 22.3 mm
- net Net-(U4-TXD): track 0.00 -> 16.8 mm
- net /EN: track 27.6 -> 44.2 mm
- net Net-(D17-K): track 0.00 -> 7.75 mm, vias 0 -> 2
- net /IO25: track 0.00 -> 4.92 mm
- net Net-(D8-K): track 0.00 -> 2.40 mm
- net /TXD0: track 0.00 -> 2.26 mm
- net /RXD0: track 0.00 -> 2.25 mm

Commit message: layout
Parts:
- moved R42 5.03 mm to (267.1, 74.1)
- moved R40 4.79 mm to (267.1, 78.9)
Routing:
- net /PA5/PH_ADC: track 0.00 -> 49.9 mm, vias 0 -> 2
- net /PA12/MAX31865_CS: track 0.00 -> 46.5 mm, vias 0 -> 4
- net /PA7/MAX31865_MISO: track 0.00 -> 46.0 mm, vias 0 -> 2
- net /PA11/MAX31865_MOSI: track 0.00 -> 44.8 mm, vias 0 -> 2
- net /PA6/MAX31865_SCK: track 0.00 -> 44.5 mm, vias 0 -> 1
- net /PB1/TDS_ADC: track 0.00 -> 43.2 mm, vias 0 -> 2
- net /PB12/RELAY1_CTRL: track 0.00 -> 38.1 mm, vias 0 -> 2
- net /PB13/RELAY2_CTRL: track 0.00 -> 35.9 mm, vias 0 -> 1
- net /PB8/RELAY5_CTRL: track 0.00 -> 35.4 mm, vias 0 -> 4
- net /PB7/SHT30_SDA: track 0.00 -> 35.1 mm, vias 0 -> 1
- net /PB14/RELAY3_CTRL: track 0.00 -> 34.7 mm, vias 0 -> 1
- net /PB15/RELAY4_CTRL: track 0.00 -> 34.1 mm, vias 0 -> 1
- net /PB9/RELAY6_CTRL: track 0.00 -> 33.9 mm, vias 0 -> 3
- net /PA2_TX/PZEM_RX: track 0.00 -> 31.9 mm, vias 0 -> 2
- net /PB6/SHT30_SCL: track 0.00 -> 31.9 mm, vias 0 -> 1
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
Commit message: hoan thanh 2 layer pcb
Routing:
- net /3.3V: track 241.1 -> 273.2 mm, vias 1 -> 6
- net /BOOT0: track 0.00 -> 21.9 mm, vias 0 -> 2
- net /BOOT1: track 0.00 -> 21.7 mm, vias 0 -> 2
- net Net-(JP2x32.1-Pin_4): track 0.00 -> 3.08 mm
- net Net-(JP2x32.1-Pin_3): track 0.00 -> 2.93 mm
- net /PB6/SHT30_SCL: track 31.9 -> 34.3 mm
- net /IO0: track 35.4 -> 37.1 mm
- net /3.3V_STM: track 67.5 -> 66.5 mm
- net /PB8/RELAY5_CTRL: track 35.4 -> 36.0 mm
- added copper zone on B.Cu, net GND
- added copper zone on F.Cu, net GND
Other:
- board outline added: 100 x 100.1 mm
